File: Nav-Lights.kicad_sch (KiCad schematic)
At the start: 0 parts

Commit message: LEDboard
Other:
- added sheet Main (main.kicad_sch)
- added sheet PCB (pcb.kicad_sch)
Changed lines of the file:
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@@
 	(generator_version "9.0")
 	(paper "A4")
+	(sheet
+		(at 63.5 74.93)
+		(size 39.37 26.67)
+		(exclude_from_sim no)
+		(in_bom yes)
+		(on_board yes)
+		(dnp no)
+		(fields_autoplaced yes)
+		(stroke
+			(width 0.1524)
+			(type solid)
+		)
+		(fill
+			(color 8 255 52 1.0000)
+		)
+		(property "Sheetname" "Main"
+			(at 63.5 74.2184 0)
+			(effects
+				(font
+					(size 5.08 5.08)
+				)
+				(justify left bottom)
+			)
+		)
+		(property "Sheetfile" "main.kicad_sch"
+			(at 63.5 102.1846 0)
+			(effects
+				(font
+					(size 1.27 1.27)
+				)
+				(justify left top)
+			)
+		)
+		(instances
+			(project "Nav-Lights"
+				(path "/30b0ade0-bb43-474b-8aae-09f32d71430b"
+					(page "2")
+				)
+			)
+		)
+	)
+	(sheet
+		(at 176.53 74.93)
+		(size 45.72 26.67)
+		(exclude_from_sim no)
+		(in_bom yes)
+		(on_board yes)
+		(dnp no)
+		(fields_autoplaced yes)
+		(stroke
+			(width 0.1524)
+			(type solid)
+		)
+		(fill
+			(color 6 253 255 1.0000)
+		)
+		(property "Sheetname" "PCB"
+			(at 176.53 74.2184 0)
+			(effects
+				(font
+					(size 5.08 5.08)
+				)
+				(justify left bottom)
+			)
+		)
+		(property "Sheetfile" "pcb.kicad_sch"
+			(at 176.53 102.1846 0)
+			(effects
+				(font
+					(size 1.27 1.27)
+				)
+				(justify left top)
+			)
+		)
+		(instances
+			(project "Nav-Lights"
+				(path "/30b0ade0-bb43-474b-8aae-09f32d71430b"
+					(page "3")
+				)
+			)
+		)
+	)
 	(sheet_instances
 		(path "/"
