File: _autosave-main.kicad_sch (KiCad schematic)
At the start: 19 parts, among them J1 Conn_01x02_Pin, U1 LMC555xCMX, U2 LT8374RUFM-WPBF

Commit message: newcircuit
Parts:
- added C10, C11, C8: C, symbol Device:C
- added C9: C_Polarized_US, symbol Device:C_Polarized_US
- added U3: TPS7B8133QDGNRQ1, VSSOP8_DGN_TEX, symbol _TPS7B81-Q1:TPS7B8133QDGNRQ1
Connections:
- net GND: now also U2.8 (GND), C10.2, C11.2, C8.2, C9.2
- net VIN: now also C8.1, C9.1
- net signal: now also U2.5 (CTRL)
- new net: C10.1, U3.1 (IN), U3.2 (EN)
- new net: U3.5 (GND), U3.6 (GND)
Other:
- moved on the sheet: C1, C2, C3, C4, C5, C6, C7, D1, D2, D3, J1, L1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
